File: GEO-HEX-1.0.0.brd (EAGLE design)
At the start: 90 x 96 mm, 127 parts

Commit message: Se organizan elementos en el Board
Se implementa toda la organización de los elementos en board. Falta incluir los opto-acopladores de comunicación entre el ADE9000 y el puerto de de E/S.
Parts:
- removed FBP5: 2 K/100Mhz, SIMI-E:L1210
- moved DP1 333.2 mm to (67.5, 80.0), flipped to the bottom, turned to 180 degrees
- moved CP3 321.8 mm to (48.0, 61.0), flipped to the bottom, turned to 90 degrees
- moved CP1 321.7 mm to (54.5, 80.0), flipped to the bottom
- moved CP4 320.0 mm to (29.0, 64.0), flipped to the bottom, turned to 90 degrees
- moved CP2 314.4 mm to (57.0, 60.0), flipped to the bottom, turned to 180 degrees
- moved LP1 305.7 mm to (65.0, 70.0), flipped to the bottom
- moved ICP2 305.2 mm to (39.0, 63.0), flipped to the bottom, turned to 270 degrees
- moved ICP1 303.2 mm to (52.0, 71.0), flipped to the bottom, turned to 270 degrees
- moved FBP3 274.2 mm to (35.0, 55.0), turned to 270 degrees
- moved FBP2 265.2 mm to (29.0, 55.0), turned to 270 degrees
- moved FBP1 264.0 mm to (22.0, 63.0), turned to 180 degrees
- moved AGND1 240.9 mm to (41.0, 46.0)
- moved CD11 230.8 mm to (30.0, 43.0), turned to 90 degrees
- moved CD6 222.9 mm to (49.0, 38.0)
- moved VCP 221.7 mm to (78.0, 83.0)
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Connections:
- new net N$1: CP1.+, ICP1.2, SP1.2
- net +3V3/A: now also FBP1.1, FBP2.1; no longer FBP5.1
- net +3V3/AA: now also FBP2.2; no longer FBP5.2
- net +3V3/D: now also FBP1.2
- net AGND: now also FBP3.2
- net GND: now also FBP3.1
- net SW: no longer CP1.+, SP1.2
