File: GEO-HEX-1.0.0.sch (EAGLE design)
At the start: 127 parts

Commit message: Se organizan elementos en el Board
Se implementa toda la organización de los elementos en board. Falta incluir los opto-acopladores de comunicación entre el ADE9000 y el puerto de de E/S.
Parts:
- removed FBP5: 2 K/100Mhz, SIMI-E:FBL1210
Connections:
- new net N$1: CP1.+, ICP1.IN, SP1.2
- net +3V3/A: now also FBP1.P$1, FBP2.P$1; no longer FBP5.P$1
- net +3V3/AA: now also FBP2.P$2; no longer FBP5.P$2
- net +3V3/D: now also FBP1.P$2
- net AGND: now also FBP3.P$2
- net GND: now also FBP3.P$1
- net SW: no longer CP1.+, SP1.2
Other:
- moved on the sheet: CP1, JP1, JP2, SP1
